File: electronics/gamepad/gamepad.kicad_pcb (KiCad board)
At the start: 2 copper layers, 8 parts, among them SW1 SMD_6x3.5mm_h2.5mm, SW2 SMD_6x3.5mm_h2.5mm, U1 ESP32-S3-WROOM-1

Commit message: initial electronics
Parts:
- added D3: White, PCM_SparkFun-LED:LED_1206_3216Metric_White, F.Cu at (185.1, 82.2)
- added D4: White, PCM_SparkFun-LED:LED_1206_3216Metric_White, F.Cu at (185.1, 85.5)
- added J1: Conn_01x04_Pin, Connector_JST:JST_XA_B04B-XASK-1-A_1x04_P2.50mm_Vertical, F.Cu at (164.8, 66.8)
- added J2: Conn_01x04_Pin, Connector_JST:JST_XA_B04B-XASK-1-A_1x04_P2.50mm_Vertical, F.Cu at (164.8, 75.3)
- added J3: Conn_01x03, PCM_SparkFun-Connector:1x03_P2.54mm, F.Cu at (177.6, 64.4)
- added J4: Conn_01x03, PCM_SparkFun-Connector:1x03_P2.54mm, F.Cu at (177.6, 68.0)
- added J5: Conn_01x03, PCM_SparkFun-Connector:1x03_P2.54mm, F.Cu at (177.6, 71.6)
- added J6: Conn_01x04, PCM_SparkFun-Connector:1x04_P2.54mm_Locking, F.Cu at (163.1, 81.3)
- added J7: Conn_01x02, PCM_SparkFun-Connector:1x02_P2.54mm, F.Cu at (184.1, 75.2)
- added J8: Conn_01x02, PCM_SparkFun-Connector:1x02_P2.54mm, F.Cu at (184.1, 78.8)
- added Q1: BC337, Package_TO_SOT_THT:TO-92_Inline, F.Cu at (177.8, 76.6)
- added Q2: BC337, Package_TO_SOT_THT:TO-92_Inline, F.Cu at (177.8, 82.4)
Connections:
- U1 pad 12: unconnected-(U1-GPIO8/TOUCH8/ADC1_CH7/SUBSPICS1-Pad12) -> /ESP_SDA
- U1 pad 15: unconnected-(U1-GPIO3/TOUCH3/ADC1_CH2-Pad15) -> /LED_BTN_LEFT
- U1 pad 16: unconnected-(U1-GPIO46-Pad16) -> /BTN_RIGHT
- U1 pad 17: unconnected-(U1-GPIO9/TOUCH9/ADC1_CH8/FSPIHD/SUBSPIHD-Pad17) -> /ESP_SCL
- U1 pad 26: unconnected-(U1-GPIO45-Pad26) -> /BTN_LEFT
- U1 pad 4: unconnected-(U1-GPIO4/TOUCH4/ADC1_CH3-Pad4) -> /LED_BTN_RIGHT
- U1 pad 5: unconnected-(U1-GPIO5/TOUCH5/ADC1_CH4-Pad5) -> /TRACKBALL_LED
- U1 pad 6: unconnected-(U1-GPIO6/TOUCH6/ADC1_CH5-Pad6) -> /HEADLIGHT_LED
- U1 pad 7: unconnected-(U1-GPIO7/TOUCH7/ADC1_CH6-Pad7) -> /BASE_LED
